File: smart-lcc.kicad_sch (KiCad schematic)
At the start: 93 parts, among them J1 280372-1, J10 Conn_01x04_Pin, J11 USB_B_Micro, J2 F0503-ZV-20-20T-R, J3 Conn_01x24, J4 BM04B-SRSS-TB(LF)(SN), J5 BM04B-SRSS-TB(LF)(SN), J6 Micro_SD_Card_Det2, J7 F0503-ZV-20-20T-R, J8 J-Link RP2040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

Commit message: WIP
Parts:
- removed C25: 22uF, 25V, X5R, Capacitor_SMD:C_0805_2012Metric, symbol Device:C_Small
- removed C26: 3300pF, 10V, X5R, Capacitor_SMD:C_0402_1005Metric, symbol Device:C_Small
- removed C27: 22uF, 10V, X5R, Capacitor_SMD:C_0805_2012Metric, symbol Device:C_Small
- removed C5, C6: 100 uF, Capacitor_THT:CP_Radial_D7.5mm_P2.50mm, symbol Device:C_Polarized_Small
- removed J10: Conn_01x04_Pin, Connector_PinHeader_2.54mm:PinHeader_1x04_P2.54mm_Vertical, symbol Connector:Conn_01x04_Pin
- removed J11: USB_B_Micro, Connector_USB:USB_Micro-B_Molex-105133-0001, symbol Connector:USB_B_Micro
- removed J7: F0503-ZV-20-20T-R, 2N7002:FPC_20, symbol Connector:Conn_01x20_Socket
- removed J8: J-Link RP2040, Connector_IDC:IDC-Header_2x10_P2.54mm_Vertical, symbol Connector_Generic:Conn_02x10_Odd_Even
- removed J9: J-Link ESP32-S3, Connector_IDC:IDC-Header_2x10_P2.54mm_Vertical, symbol Connector_Generic:Conn_02x10_Odd_Even
- removed JP1: Jumper_2_Bridged, Connector_PinHeader_2.54mm:PinHeader_1x02_P2.54mm_Vertical, symbol Jumper:Jumper_2_Bridged
- removed R12: 1M21, Resistor_SMD:R_0402_1005Metric, symbol Device:R_Small
- removed R13: 383K, Resistor_SMD:R_0402_1005Metric, symbol Device:R_Small
- removed SW3, SW4, SW5: SW_Push, SW_Push_ADTSMW65:ADTSMW65, symbol Switch:SW_Push
- removed U1: PTN04050C, Module:Texas_EUS_R-PDSS-T5_THT, symbol Converter_DCDC:PTN78000H_EUS-5
- removed U6: LMZ21701SILR, LMZ21701SILR:CONV_LMZ21701SILR, symbol LMZ21701SILR:LMZ21701SILR
- added C5, C6: NC, Capacitor_SMD:C_0402_1005Metric, symbol Device:C_Small
- added JP1: SolderJumper_3_Bridged12, Jumper:SolderJumper-3_P1.3mm_Bridged2Bar12_RoundedPad1.0x1.5mm_NumberLabels, symbol Jumper:SolderJumper_3_Bridged12
- added Q3: 2N7002, Package_TO_SOT_SMD:SOT-23, symbol Transistor_FET:2N7002
- added R14: 0R, Resistor_SMD:R_0402_1005Metric, symbol Device:R_Small
- added U1, U6: MAX40200AUK, Package_TO_SOT_SMD:SOT-23-5, symbol Analog_Switch:MAX40200AUK
- added U8: LM5050-1, Package_TO_SOT_SMD:TSOT-23-6, symbol Power_Management:LM5050-1
- J1: footprint TE_280372-1 -> 280372-1:TE_280372-1
- R7: value 1K33, 0.01W, 1% -> 0R; footprint Resistor_THT:R_Axial_DIN0204_L3.6mm_D1.6mm_P7.62mm_Horizontal -> Resistor_SMD:R_0402_1005Metric; JLCPCB Basic (none) -> N; LCSC (none) -> C3017451
Connections:
- net +3V3: now also JP1.3 (B), U1.5 (OUT); no longer C4.1, J3.5 (Pin_5), TP16.1
- net 3V3_MCU: now also U1.1 (VDD), U1.3 (EN)
- net 3V3_OLED: now also U6.1 (VDD), U6.3 (EN)
- net GND: now also C5.2, C6.1, JP1.1 (A), U1.2 (GND), U6.2 (GND), U8.2 (GND); no longer J2.2 (Pin_2), U3.15 (GPIO3/TOUCH3/ADC1_CH2)
- net RP2040_ESP32_CTS: now also U3.22 (GPIO14/TOUCH14/ADC2_CH3/FSPIWP/FSPIDQS/SUBSPIWP); no longer U3.13 (GPIO19/U1RTS/ADC2_CH8/CLK_OUT2/USB_D-)
- net RP2040_ESP32_RTS: now also U3.21 (GPIO13/TOUCH13/ADC2_CH2/FSPIQ/FSPIIO7/SUBSPIQ); no longer U3.14 (GPIO20/U1CTS/ADC2_CH9/CLK_OUT1/USB_D+)
- net RP2040_ESP32_RX: no longer J2.10 (Pin_10)
- net RP2040_ESP32_TX: no longer J2.9 (Pin_9)
- net ESP32_USB_DP: now reaches R7.1
- net ESP32_USB_DP: now also J2.9 (Pin_9), C6.2
- net +12V renamed 12V_OLED_SAFE
- net 12V_OLED_SAFE: now also Q3.3 (D), U8.1 (VS), U8.6 (OUT); no longer J1.1
- net GND2 renamed ESP32_USB_PRE_R_DP
- net ESP32_USB_PRE_R_DP: now also U3.14 (GPIO20/U1CTS/ADC2_CH9/CLK_OUT1/USB_D+)
- new net: JP1.2 (C), U3.15 (GPIO3/TOUCH3/ADC1_CH2)
- new net: Q3.1 (G), U8.5 (GATE)
- new net 12V_OLED: J1.1, Q3.2 (S), U8.4 (IN)
- new net 3V3_OLED_SAFE: C4.1, J2.2 (Pin_2), J3.5 (Pin_5), TP16.1, U6.5 (OUT)
- new net ESP32_USB_DN: C5.1, J2.10 (Pin_10), R14.1
- new net ESP32_USB_PRE_R_DN: R14.2, U3.13 (GPIO19/U1RTS/ADC2_CH8/CLK_OUT2/USB_D-)
- no-connect marks 32 -> 20
Other:
- note added: "Power handling"
- note removed: "Debug Power Supply (Daughter Board) (v)"
- note removed: "Debug daughter board connector (Daughter board) (v)"
- note removed: "Debug push buttons (Daughter Board) (v)"
- note removed: "Power Supply (v)"
- note removed: "SWD/JTAG Connectors (Daughter board) (v)"
- note removed: "USB/UART connectors (Daughter Board) (v)"
