File: smart-lcc.kicad_sch (KiCad schematic)
At the start: 117 parts, among them J1 280372-1, J2 F0503-ZV-24-20T-R, J3 Conn_01x24, J4 BM04B-SRSS-TB(LF)(SN), J5 BM04B-SRSS-TB(LF)(SN), J6 Micro_SD_Card_Det2, J7 Conn_01x12, J8 BM04B-SRSS-TB(LF)(SN), Q1 2N7002, Q2 2N7002, Q4 2N7002, Q6 NTGD3148NT1G, SW1 SW_Push, SW2 SW_Push, U1 LM5050-1, U2 RP2040, U3 ESP32-S3-WROOM-1, U4 W25Q16JVSNIQ (Program Flash), U5 W25Q16JVSNIQ (Opt. Settings f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, U6 TPS82130, U7 74LVC1G125, U8 LM5050-1, Y1 XYDBPCNANF-12MHZ

Commit message: R3A (preliminary)
Changes:
* Switched the OLED connector for an EyeSPI connector (feature parity with APEC)
* Removed the need for a debug board by moving USB connectors and SWD/JTAG ports to this board
* Move to 6 layers
* Component changes for a more dense design
Parts:
- removed C1, C3: 2.2 µF / 25V, Capacitor_SMD:C_0603_1608Metric, symbol Device:C_Small
- removed C4: 1 uF, 16V, Capacitor_SMD:C_0402_1005Metric, symbol Device:C_Small
- removed J2: F0503-ZV-24-20T-R, FlexibleFPC:Flexible24Pin, symbol Connector:Conn_01x24_Socket
- removed J3: Conn_01x24, FH34SRJ-24S-0.5SH_50:FH34SRJ24S05SH50, symbol Connector_Generic:Conn_01x24
- removed J7: Conn_01x12, TFT_1.47IN_172X320_12P:TFT_1.47IN_172X320_12P, symbol Connector_Generic:Conn_01x12
- removed Q4: 2N7002, Package_TO_SOT_SMD:SOT-23, symbol Transistor_FET:2N7002
- removed R1: 910K, Resistor_SMD:R_0402_1005Metric, symbol Device:R
- removed R18: 10R, Resistor_SMD:R_0402_1005Metric, symbol Device:R_Small
- removed TP1, TP10, TP2, TP28, TP29, TP3, TP4, TP5, TP6, TP7, TP8, TP9: TestPoint_Small, TestPoint:TestPoint_Pad_D1.0mm, symbol Connector:TestPoint_Small
- removed TP13, TP17, TP18: TestPoint, TestPoint:TestPoint_Pad_D1.0mm, symbol Connector:TestPoint
- removed TP14, TP15, TP16, TP19: TestPoint, TestPoint:TestPoint_Pad_D1.5mm, symbol Connector:TestPoint
- removed TP20, TP21, TP22, TP23, TP24, TP25, TP26, TP27: TestPoint_Small, TestPoint:TestPoint_Pad_D1.5mm, symbol Connector:TestPoint_Small
- added J10, J7: Conn_02x05_Odd_Even, Connector_PinHeader_1.27mm:PinHeader_2x05_P1.27mm_Vertical_SMD, symbol Connector_Generic:Conn_02x05_Odd_Even
- added J11: Conn_02x03_Odd_Even, Connector_PinHeader_1.27mm:PinHeader_2x03_P1.27mm_Vertical_SMD, symbol Connector_Generic:Conn_02x03_Odd_Even
- added J12: Conn_01x12, TFT_1.47IN_172X320_12P:TFT_1.47IN_172X320_12P, symbol Connector_Generic:Conn_01x12
- added J2, J3: USB_B_Micro, Connector_USB:USB_Micro-B_Molex-105133-0001, symbol Connector:USB_B_Micro
- added J9: Molex_0525591853, Molex_5051101892:CON_5051101892_MOL, symbol ADS1119:EyeSPI
- added Q3: 2N7002, Package_TO_SOT_SMD:SOT-23, symbol Transistor_FET:2N7002
- added Q4: DMN63D8LDW, PCM_Package_TO_SOT_SMD_AKL:SOT-363_SC-70-6, symbol PCM_Transistor_MOSFET_AKL:DMN63D8LDW
- added R1: 100R, Resistor_SMD:R_0201_0603Metric, symbol Device:R_Small
- added R18: 4K7, Resistor_SMD:R_0201_0603Metric, symbol Device:R
- added SW3, SW4, SW5, SW6: SW_Push, ul_PTS815-SJM-250-SMTR-LFS:SW4_PTS815 SJM 250 SMTR LFS_CNK, symbol Switch:SW_Push
- added TP1, TP2, TP3, TP4: TestPoint, TestPoint:TestPoint_Pad_D1.5mm, symbol Connector:TestPoint
- C10, C13, C14, C15, C16, C17, C18, C19, C20, C21, C22, C24, C9: footprint Capacitor_SMD:C_0402_1005Metric -> Capacitor_SMD:C_0201_0603Metric; Comment 16 V, X5R, 0201 is C467016 -> (none); LCSC C960916 -> C412246
- C11, C12, C23, C8: value 1 uF, 16V -> 1 uF, 10V; footprint Capacitor_SMD:C_0402_1005Metric -> Capacitor_SMD:C_0201_0603Metric; Comment 16 V, X5R -> (none); LCSC C268023 -> C426073
- R10, R11, R13, R14, R15, R16, R17, R19, R2, R20, R21, R22, R23, R24, R25, R26, R27, R3, R4, R5, R6, R7, R8, R9: footprint Resistor_SMD:R_0402_1005Metric -> Resistor_SMD:R_0201_0603Metric
- R12: value 100R -> 10R; footprint Resistor_SMD:R_0402_1005Metric -> Resistor_SMD:R_0201_0603Metric; LCSC C2935235 -> C851817
- U4, U5: footprint PCM_Package_SO_AKL:SOIC-8_3.9x4.9mm_P1.27mm -> W25Q16JVUXIQ:SON50P300X200X60-9N; LCSC C115407 -> C2843335
Connections:
- net ESP32_CTS0 is gone; now on net SSD1309_RES: U3.9 (GPIO16/U0CTS/ADC2_CH5/XTAL_32K_N)
- net ESP32_RTS0 is gone; now on net SSD1309_DC: U3.8 (GPIO15/U0RTS/ADC2_CH4/XTAL_32K_P)
- net +3V3: now also R12.1, J10.1 (Pin_1), J12.4 (Pin_4), J7.1 (Pin_1), J9.1 (Vcc)
- net BACKLIGHT: now also J9.2 (BACKLIGHT), Q3.1 (G)
- net ESP32_EN: now also J10.10 (Pin_10), J11.1 (Pin_1), SW6.1
- net ESP32_GPIO0: now also J11.6 (Pin_6), R1.1, SW5.1
- net ESP32_GPIO45: now also J9.18 (GPIO2)
- net ESP32_GPIO46: now also J9.17 (GPIO1)
- net ESP32_QWIIC_SCL: now also J9.13 (SCL)
- net ESP32_QWIIC_SDA: now also J9.14 (SDA)
- net ESP32_RXD0: now also J11.3 (Pin_3)
- net ESP32_TCK: now also J10.4 (Pin_4)
- net ESP32_TDI: now also J10.8 (Pin_8)
- net ESP32_TDO: now also J10.6 (Pin_6)
- net ESP32_TMS: now also J10.2 (Pin_2)
- net ESP32_TXD0: now also J11.5 (Pin_5)
- net ESP32_USB_DN: now also J3.2 (D-)
- net ESP32_USB_DP: now also J3.3 (D+)
- net GND: now also J10.3 (Pin_3), J10.5 (Pin_5), J10.9 (Pin_9), J11.4 (Pin_4), J12.1 (Pin_1), J12.12 (Pin_12), J12.5 (Pin_5), J12.6 (Pin_6), J2.5 (GND), J2.6 (Shield), J3.5 (GND), J3.6 (Shield), J7.3 (Pin_3), J7.5 (Pin_5), J7.9 (Pin_9), J9.3 (GND), Q3.2 (S), Q4.1 (S1), Q4.4 (S2), R18.2, SW3.2, SW4.2, SW5.2, SW6.2
- net RP2040_BOOTSEL: now also Q4.6 (D1), SW3.1; no longer U3.5 (GPIO5/TOUCH5/ADC1_CH4)
- net RP2040_ESP32_RX: now also U3.11 (GPIO18/U1RXD/ADC2_CH7/CLK_OUT3); no longer U3.10 (GPIO17/U1TXD/ADC2_CH6)
- net RP2040_ESP32_TX: now also U3.12 (GPIO8/TOUCH8/ADC1_CH7/SUBSPICS1); no longer U3.11 (GPIO18/U1RXD/ADC2_CH7/CLK_OUT3)
- net RP2040_RESETn: now also J7.10 (Pin_10), Q4.3 (D2), SW4.1; no longer R11.1, U3.4 (GPIO4/TOUCH4/ADC1_CH3)
- net RP2040_SERIAL_BOOT: now also U3.17 (GPIO9/TOUCH9/ADC1_CH8/FSPIHD/SUBSPIHD); no longer U3.6 (GPIO6/TOUCH6/ADC1_CH5)
- net RP2040_SET_CS: now also U2.18 (GPIO15); no longer U2.28 (GPIO17)
- net RP2040_SWCLK: now also J7.4 (Pin_4)
- net RP2040_SWD: now also J7.2 (Pin_2)
- net RP2040_USB_DN: now also J2.2 (D-)
- net RP2040_USB_DP: now also J2.3 (D+)
- net SSD1309_CS: now also U3.10 (GPIO17/U1TXD/ADC2_CH6), J12.8 (Pin_8), J9.9 (DISP_CS); no longer U3.18 (GPIO10/TOUCH10/ADC1_CH9/FSPICS0/FSPIIO4/SUBSPICS0)
- net SSD1309_DC: now also J12.7 (Pin_7), J9.7 (DC); no longer U3.17 (GPIO9/TOUCH9/ADC1_CH8/FSPIHD/SUBSPIHD)
- net SSD1309_MOSI: now also U3.6 (GPIO6/TOUCH6/ADC1_CH5), J12.10 (Pin_10), J9.5 (MOSI); no longer U3.19 (GPIO11/TOUCH11/ADC2_CH0/FSPID/FSPIIO5/SUBSPID)
- net SSD1309_RES: now also J12.11 (Pin_11), J9.8 (RESET); no longer U3.12 (GPIO8/TOUCH8/ADC1_CH7/SUBSPICS1)
- net SSD1309_SCLK: now also U3.5 (GPIO5/TOUCH5/ADC1_CH4), J12.9 (Pin_9), J9.4 (SCK); no longer U3.20 (GPIO12/TOUCH12/ADC2_CH1/FSPICLK/FSPIIO6/SUBSPICLK)
- net VIN_DEBUG: now also J11.2 (Pin_2), J2.1 (VBUS), J3.1 (VBUS)
- net ESP32_EYESPI_BUSY_TE: now reaches U3.25 (GPIO48/SPICLK_N/SUBSPICLK_N_DIFF)
- net ESP32_EYESPI_BUSY_TE: now also J9.16 (BUSY/TE); no longer R12.1
- net ESP32_GPIO7: now reaches U3.7 (GPIO7/TOUCH7/ADC1_CH6)
- net ESP32_GPIO7: now also J9.6 (MISO)
- net at R12.2: now also J12.3 (Pin_3); no longer D4.2 (A)
- net 12V_OLED renamed VIN_CONN
- net RP2040_ESP32_CTS: no longer names the net of U2.4 (GPIO2)
- net RP2040_ESP32_CTS: no longer U3.22 (GPIO14/TOUCH14/ADC2_CH3/FSPIWP/FSPIDQS/SUBSPIWP)
- net RP2040_ESP32_RTS: no longer names the net of U2.5 (GPIO3)
- net RP2040_ESP32_RTS: no longer U3.21 (GPIO13/TOUCH13/ADC2_CH2/FSPIQ/FSPIIO7/SUBSPIQ)
- new net: J12.2 (Pin_2), Q3.3 (D)
- new net: D4.2 (A), R1.2
- new net ESP32_BOOTSEL_RP2040: Q4.2 (G1), R11.1, U3.18 (GPIO10/TOUCH10/ADC1_CH9/FSPICS0/FSPIIO4/SUBSPICS0)
- new net ESP32_DISABLE_RP2040: Q4.5 (G2), R18.1, U3.4 (GPIO4/TOUCH4/ADC1_CH3)
- new net ESP32_EYESPI_INT: J9.15 (INT), U3.22 (GPIO14/TOUCH14/ADC2_CH3/FSPIWP/FSPIDQS/SUBSPIWP)
- new net ESP32_EYESPI_MEM_CS: J9.11 (MEM_CS), U3.20 (GPIO12/TOUCH12/ADC2_CH1/FSPICLK/FSPIIO6/SUBSPICLK)
- new net ESP32_EYESPI_SD_CS: J9.10 (SD_CS), U3.19 (GPIO11/TOUCH11/ADC2_CH0/FSPID/FSPIIO5/SUBSPID)
- new net ESP32_EYESPI_TS_CS: J9.12 (TS_CS), U3.21 (GPIO13/TOUCH13/ADC2_CH2/FSPIQ/FSPIIO7/SUBSPIQ)
- no-connect marks 10 -> 14
